Commit message: started on the gazebo tutorials

File: src/scara_setup_description/urdf/scara_setup.urdf (robot description, URDF)
Before this commit: robot scara_setup, 6 links, 5 joints
Links:
- added link effector_tip
- added link mount_point
- link Arm: geometry collision mesh filename=package://scara_setup_description/meshes/Arm.STL; visual mesh filename=package://scara_setup_description/meshes/Arm.STL
- link Cart: geometry collision mesh filename=package://scara_setup_description/meshes/Cart.STL; visual mesh filename=package://scara_setup_description/meshes/Cart.STL
- link Finger: geometry collision mesh filename=package://scara_setup_description/meshes/Finger.STL; visual mesh filename=package://scara_setup_description/meshes/Finger.STL
- link ForeArm: geometry collision mesh filename=package://scara_setup_description/meshes/ForeArm.STL; visual mesh filename=package://scara_setup_description/meshes/ForeArm.STL
- link Hand: geometry collision mesh filename=package://scara_setup_description/meshes/Hand.STL; visual mesh filename=package://scara_setup_description/meshes/Hand.STL
- link frame: geometry collision mesh filename=package://scara_setup_description/meshes/base_link.STL; visual mesh filename=package://scara_setup_description/meshes/base_link.STL
Joints:
- added joint dummy: type fixed, parent mount_point, child frame, origin xyz=0 0 0 rpy=0 0 0
- added joint tip_joint: type fixed, parent Finger, child effector_tip, origin xyz=0.0665 0 0 rpy=1.57 0 0

Commit message: Edited the model files (taking rrbots files as a base) controllers remain not working, however, the model and controllers spawn correctly

File: src/scara_setup_description/urdf/scara_setup.urdf (robot description, URDF)
Before this commit: robot scara_setup, 8 links, 7 joints
Links:
- added link world
Joints:
- added joint fixed: type fixed, parent world, child mount_point, origin xyz=0 0 0.3 rpy=0 0 0

Commit message: MoveIt now working with Gazebo. Current problems: - PID controllers relatively weak (or the arm relatively heavy) - Linear axis not going up fully - Some warnings remain
Issue #65

File: src/scara_setup_description/urdf/scara_setup.urdf (robot description, URDF)
Before this commit: robot scara_setup, 9 links, 8 joints
Links:
- removed link Arm
- removed link Cart
- removed link Finger
- removed link ForeArm
- removed link Hand
- added link arm, mass 0.313727406555667; collision mesh filename=package://scara_setup_description/meshes/arm.STL; visual mesh filename=package://scara_setup_description/meshes/arm.STL
- added link cart, mass 0.571810586822584; collision mesh filename=package://scara_setup_description/meshes/cart.STL; visual mesh filename=package://scara_setup_description/meshes/cart.STL
- added link finger, mass 0.18562; collision mesh filename=package://scara_setup_description/meshes/finger.STL; visual mesh filename=package://scara_setup_description/meshes/finger.STL
- added link forearm, mass 0.46163; collision mesh filename=package://scara_setup_description/meshes/forearm.STL; visual mesh filename=package://scara_setup_description/meshes/forearm.STL
- added link hand, mass 0.281; collision mesh filename=package://scara_setup_description/meshes/hand.STL; visual mesh filename=package://scara_setup_description/meshes/hand.STL
Joints:
- removed joint Elbow
- removed joint FingerJoint
- removed joint Linear
- removed joint Shoulder
- removed joint Wrist
- added joint elbow: type revolute, parent arm, child forearm, origin xyz=-0.35 0 0 rpy=7.3171E-17 -1.0978 1.5708, axis -0.45558 0 0.8902, limit lower=-2.36 upper=2.36 effort=1.0 velocity=1.0
- added joint fingerjoint: type revolute, parent hand, child finger, origin xyz=-0.12711 0.0285 0 rpy=-1.5708 -6.123E-17 3.1416, axis 0 1 0, limit lower=-1.57 upper=1.57 effort=1.0 velocity=1.0
- added joint linear: type prismatic, parent frame, child cart, origin xyz=0 -0.0185 0.08 rpy=3.1416 0 0, axis 0 0 -1, limit lower=0 upper=0.5 effort=1000.0 velocity=10.0
- added joint shoulder: type revolute, parent cart, child arm, origin xyz=0 0.094508 0.0285 rpy=-1.5708 0 -1.5708, axis 0 -1 0, limit lower=-1.57 upper=1.57 effort=1.0 velocity=1.0
- added joint wrist: type revolute, parent forearm, child hand, origin xyz=0.022096 0.37901 -0.043174 rpy=-1.0978 -1.5187E-17 -1.5708, axis 0 -1 0, limit lower=-2.36 upper=2.36 effort=1.0 velocity=1.0
- joint tip_joint: parent Finger -> finger

Commit message: Edited the model and controllers, now acts like a servo based arm

File: src/scara_setup_description/urdf/scara_setup.urdf (robot description, URDF)
Before this commit: robot scara_setup, 9 links, 8 joints
Links:
- link arm: mass 0.313727406555667 -> 0.81408
- link cart: mass 0.571810586822584 -> 1.2438
- link forearm: mass 0.46163 -> 1.2068
- link frame: mass 1.493046 -> 1.493
- link hand: mass 0.281 -> 0.74303
Joints:
- joint elbow: limit lower=-2.36 upper=2.36 effort=1.0 velocity=1.0 -> lower=-2.35 upper=2.35 effort=6 velocity=198
- joint fingerjoint: limit lower=-1.57 upper=1.57 effort=1.0 velocity=1.0 -> lower=-1.57 upper=1.57 effort=1.5 velocity=370
- joint linear: limit lower=0 upper=0.5 effort=1000.0 velocity=10.0 -> lower=0 upper=0.424 effort=500 velocity=0.3; origin xyz=0 -0.0185 0.08 rpy=3.1416 0 0 -> xyz=0 -0.0185 0.049 rpy=3.1416 0 0
- joint shoulder: limit lower=-1.57 upper=1.57 effort=1.0 velocity=1.0 -> lower=-2.35 upper=2.35 effort=6 velocity=198
- joint wrist: limit lower=-2.36 upper=2.36 effort=1.0 velocity=1.0 -> lower=-2.35 upper=2.35 effort=6 velocity=198

Commit message: Wrist control working, editted topics in HWA, editted joint limits in URDF

File: src/scara_setup_description/urdf/scara_setup.urdf (robot description, URDF)
Before this commit: robot scara_setup, 9 links, 8 joints
Joints:
- joint elbow: limit lower=-2.35 upper=2.35 effort=6 velocity=198 -> lower=-1.57 upper=1.57 effort=6 velocity=198
- joint shoulder: limit lower=-2.35 upper=2.35 effort=6 velocity=198 -> lower=-1.57 upper=1.57 effort=6 velocity=198
- joint wrist: limit lower=-2.35 upper=2.35 effort=6 velocity=198 -> lower=-1.57 upper=1.57 effort=6 velocity=198

Commit message: Editted the URDF model (now proper arm lengths) Inverted the motors to go with the URDF change Now able to plan & execute trajectories on physical arm

File: src/scara_setup_description/urdf/scara_setup.urdf (robot description, URDF)
Before this commit: robot scara_setup, 9 links, 8 joints
Links:
- link cart: mass 1.2438 -> 1.2925
- link forearm: mass 1.2068 -> 1.2555
- link hand: mass 0.74303 -> 0.79174
Joints:
- joint elbow: axis -0.45558 0 0.8902 -> 0 1 0; origin xyz=-0.35 0 0 rpy=7.3171E-17 -1.0978 1.5708 -> xyz=-0.35 0.0015 0 rpy=3.1416 -1.2246E-16 3.1416
- joint fingerjoint: axis 0 1 0 -> 0 -1 0; origin xyz=-0.12711 0.0285 0 rpy=-1.5708 -6.123E-17 3.1416 -> xyz=-0.15461 0.027 -0.02 rpy=-1.5708 -6.123E-17 3.1416
- joint linear: origin xyz=0 -0.0185 0.049 rpy=3.1416 0 0 -> xyz=0 -0.0185 0.049001 rpy=3.1416 0 0
- joint shoulder: axis 0 -1 0 -> 0 1 0; origin xyz=0 0.094508 0.0285 rpy=-1.5708 0 -1.5708 -> xyz=0 0.11051 0.0285 rpy=-1.5708 0 -1.5708
- joint wrist: axis 0 -1 0 -> 0 1 0; origin xyz=0.022096 0.37901 -0.043174 rpy=-1.0978 -1.5187E-17 -1.5708 -> xyz=0.42501 0.0485 0 rpy=3.1416 1.2246E-16 3.1416

Commit message: updated the URDF model, joint coordinate systems are now defined

File: src/scara_setup_description/urdf/scara_setup.urdf (robot description, URDF)
Before this commit: robot scara_setup, 9 links, 8 joints
Links:
- link frame: geometry collision mesh filename=package://scara_setup_description/meshes/frame.STL; visual mesh filename=package://scara_setup_description/meshes/frame.STL
Joints:
- joint elbow: axis 0 1 0 -> 0 0 1; limit lower=-1.57 upper=1.57 effort=6 velocity=198 -> lower=-1.57 upper=1.57 effort=6 velocity=3.295; origin xyz=-0.35 0.0015 0 rpy=3.1416 -1.2246E-16 3.1416 -> xyz=0 0.35 0 rpy=6.9389E-16 -2.0817E-15 -1.4444E-30
- joint fingerjoint: axis 0 -1 0 -> -1 0 0; limit lower=-1.57 upper=1.57 effort=1.5 velocity=370 -> lower=-1.57 upper=1.57 effort=1.5 velocity=370.7; origin xyz=-0.15461 0.027 -0.02 rpy=-1.5708 -6.123E-17 3.1416 -> xyz=0 0.14311 0.0285 rpy=0 -1.3878E-15 0
- joint linear: axis 0 0 -1 -> 0 0 1; limit lower=0 upper=0.424 effort=500 velocity=0.3 -> lower=0 upper=0.424 effort=501 velocity=0.0063; origin xyz=0 -0.0185 0.049001 rpy=3.1416 0 0 -> xyz=0 0.0159 0.049 rpy=1.3878E-15 -1.3878E-15 -7.9703E-17
- joint shoulder: axis 0 1 0 -> 0 0 1; limit lower=-1.57 upper=1.57 effort=6 velocity=198 -> lower=-1.57 upper=1.57 effort=6 velocity=3.295; origin xyz=0 0.11051 0.0285 rpy=-1.5708 0 -1.5708 -> xyz=0 0.11311 -0.0285 rpy=-1.3878E-15 1.3878E-15 7.9703E-17
- joint tip_joint: origin xyz=0.0665 0 0 rpy=1.57 0 0 -> xyz=0 0.0665 0 rpy=0 0 0
- joint wrist: axis 0 1 0 -> 0 0 1; limit lower=-1.57 upper=1.57 effort=6 velocity=198 -> lower=-1.57 upper=1.57 effort=6 velocity=3.295; origin xyz=0.42501 0.0485 0 rpy=3.1416 1.2246E-16 3.1416 -> xyz=0 0.42501 0.0485 rpy=-6.9389E-16 2.0817E-15 0

Commit message: add tf support capturing /world to /camera_base_link

File: src/scara_setup_description/urdf/scara_setup.urdf (robot description, URDF)
Before this commit: robot scara_setup, 9 links, 8 joints
Joints:
- joint elbow: limit lower=-1.57 upper=1.57 effort=6 velocity=3.295 -> lower=-2.57 upper=2.57 effort=6 velocity=3.295
- joint fingerjoint: limit lower=-1.57 upper=1.57 effort=1.5 velocity=370.7 -> lower=-2.57 upper=2.57 effort=1.5 velocity=370.7
- joint shoulder: limit lower=-1.57 upper=1.57 effort=6 velocity=3.295 -> lower=-2.57 upper=2.57 effort=6 velocity=3.295
- joint wrist: limit lower=-1.57 upper=1.57 effort=6 velocity=3.295 -> lower=-2.57 upper=2.57 effort=6 velocity=3.295

Commit message: test version

File: src/scara_setup_description/urdf/scara_setup.urdf (robot description, URDF)
Before this commit: robot scara_setup, 9 links, 8 joints
Joints:
- joint elbow: limit lower=-2.57 upper=2.57 effort=6 velocity=3.295 -> lower=-1.57 upper=1.57 effort=6 velocity=3.295
- joint shoulder: limit lower=-2.57 upper=2.57 effort=6 velocity=3.295 -> lower=-1.57 upper=1.57 effort=6 velocity=3.295
- joint wrist: limit lower=-2.57 upper=2.57 effort=6 velocity=3.295 -> lower=-1.57 upper=1.57 effort=6 velocity=3.295

Commit message: Changed joints to use absolute encoders. CONTROL IS UNTUNED, UNSTABLE OPERATION

File: src/scara_setup_description/urdf/scara_setup.urdf (robot description, URDF)
Before this commit: robot scara_setup, 9 links, 8 joints
Joints:
- joint shoulder: limit lower=-1.57 upper=1.57 effort=6 velocity=3.295 -> lower=-1.9 upper=1.9 effort=6 velocity=3.295
- joint wrist: limit lower=-1.57 upper=1.57 effort=6 velocity=3.295 -> lower=-1.9 upper=1.9 effort=6 velocity=3.295

Commit message: Made some changes to the control loops for velocity based joints. CURRENTLY UNSTABLE

File: src/scara_setup_description/urdf/scara_setup.urdf (robot description, URDF)
Before this commit: robot scara_setup, 9 links, 8 joints
Joints:
- joint elbow: limit lower=-1.57 upper=1.57 effort=6 velocity=3.295 -> lower=-1.57 upper=1.57 effort=6 velocity=6.106
- joint shoulder: limit lower=-1.9 upper=1.9 effort=6 velocity=3.295 -> lower=-1.9 upper=1.9 effort=6 velocity=6.106
- joint wrist: limit lower=-1.9 upper=1.9 effort=6 velocity=3.295 -> lower=-1.9 upper=1.9 effort=6 velocity=6.106
